Commit message: move finger mesh origin to tip of the finger

File: robotiq_description/urdf/hand_e/hand_e_macro.ros2_control.xacro (robot description, xacro)
@@ -6,5 +6,5 @@
                fake_sensor_commands:=false"
                >
-    <ros2_control name="robotiq_hand_e_ros2_control" type="system">
+    <ros2_control name="RobotiqHandE_HardwareInterface" type="system">
       <hardware>
         <xacro:if value="${use_fake_hardware}">

File: robotiq_description/urdf/hand_e/hand_e_macro.xacro (robot description, xacro)
@@ -22,10 +22,10 @@
       <visual>
         <geometry>
-          <mesh filename="package://robotiq_description/meshes/hand_e/visual/finger_1.dae"/>
+          <mesh filename="package://robotiq_description/meshes/hand_e/visual/finger_left.dae"/>
         </geometry>
       </visual>
       <collision>
         <geometry>
-          <mesh filename="package://robotiq_description/meshes/hand_e/collision/finger_1.dae"/>
+          <mesh filename="package://robotiq_description/meshes/hand_e/collision/finger_left.dae"/>
         </geometry>
       </collision>
@@ -34,10 +34,10 @@
       <visual>
         <geometry>
-          <mesh filename="package://robotiq_description/meshes/hand_e/visual/finger_2.dae"/>
+          <mesh filename="package://robotiq_description/meshes/hand_e/visual/finger_right.dae"/>
         </geometry>
       </visual>
       <collision>
         <geometry>
-          <mesh filename="package://robotiq_description/meshes/hand_e/collision/finger_2.dae"/>
+          <mesh filename="package://robotiq_description/meshes/hand_e/collision/finger_right.dae"/>
         </geometry>
       </collision>
@@ -49,5 +49,5 @@
     </joint>
     <joint name="${prefix}robotiq_hand_e_left_finger_joint" type="prismatic">
-      <origin xyz="0 0 0.099" rpy="0 0 0"/>
+      <origin xyz="0 0 ${0.099 + 0.047}" rpy="0 0 0"/>
       <parent link="${prefix}robotiq_hand_e_base_link"/>
       <child link="${prefix}robotiq_hand_e_left_finger"/>
@@ -56,5 +56,5 @@
     </joint>
     <joint name="${prefix}robotiq_hand_e_right_finger_joint" type="prismatic">
-      <origin xyz="0 0 0.099" rpy="0 0 0"/>
+      <origin xyz="0 0 ${0.099 + 0.047}" rpy="0 0 0"/>
       <parent link="${prefix}robotiq_hand_e_base_link"/>
       <child link="${prefix}robotiq_hand_e_right_finger"/>
