Commit message: add gripper collision meshes

File: robotiq_description/urdf/hand_e/hand_e_macro.xacro (robot description, xacro)
@@ -9,25 +9,37 @@
     <link name="${prefix}robotiq_hand_e_base_link">
       <visual>
-        <origin xyz="0 0 0" rpy="0 0 0" />
         <geometry>
           <mesh filename="package://robotiq_description/meshes/hand_e/visual/hand_e.dae"/>
         </geometry>
       </visual>
+      <collision>
+        <geometry>
+          <mesh filename="package://robotiq_description/meshes/hand_e/collision/hand_e.dae"/>
+        </geometry>
+      </collision>
     </link>
     <link name="${prefix}robotiq_hand_e_left_finger">
       <visual>
-        <origin xyz="0 0 0" rpy="0 0 0" />
         <geometry>
           <mesh filename="package://robotiq_description/meshes/hand_e/visual/finger_1.dae"/>
         </geometry>
       </visual>
+      <collision>
+        <geometry>
+          <mesh filename="package://robotiq_description/meshes/hand_e/collision/finger_1.dae"/>
+        </geometry>
+      </collision>
     </link>
     <link name="${prefix}robotiq_hand_e_right_finger">
       <visual>
-        <origin xyz="0 0 0" rpy="0 0 0" />
         <geometry>
           <mesh filename="package://robotiq_description/meshes/hand_e/visual/finger_2.dae"/>
         </geometry>
       </visual>
+      <collision>
+        <geometry>
+          <mesh filename="package://robotiq_description/meshes/hand_e/collision/finger_2.dae"/>
+        </geometry>
+      </collision>
     </link>
     <joint name="${prefix}robotiq_hand_e_base_joint" type="fixed">

Commit message: specify correct movement axis

File: robotiq_description/urdf/hand_e/hand_e_macro.xacro (robot description, xacro)
@@ -52,5 +52,5 @@
       <parent link="${prefix}robotiq_hand_e_base_link"/>
       <child link="${prefix}robotiq_hand_e_left_finger"/>
-      <axis xyz="0 -1 0"/>
+      <axis xyz="-1 0 0"/>
       <limit effort="130" lower="0" upper="0.025" velocity="0.15"/>
     </joint>
@@ -59,5 +59,5 @@
       <parent link="${prefix}robotiq_hand_e_base_link"/>
       <child link="${prefix}robotiq_hand_e_right_finger"/>
-      <axis xyz="0 1 0"/>
+      <axis xyz="1 0 0"/>
       <limit effort="130" lower="0" upper="0.025" velocity="0.15"/>
       <mimic joint="${prefix}robotiq_hand_e_left_finger_joint" multiplier="1" offset="0"/>

Commit message: ensure we start at joint state open=0.0, and that close=0.025

File: robotiq_description/urdf/hand_e/hand_e_macro.xacro (robot description, xacro)
@@ -49,15 +49,15 @@
     </joint>
     <joint name="${prefix}robotiq_hand_e_left_finger_joint" type="prismatic">
-      <origin xyz="0 0 ${0.099 + 0.047}" rpy="0 0 0"/>
+      <origin xyz="-0.025 0 ${0.099 + 0.047}" rpy="0 0 0"/>
       <parent link="${prefix}robotiq_hand_e_base_link"/>
       <child link="${prefix}robotiq_hand_e_left_finger"/>
-      <axis xyz="-1 0 0"/>
+      <axis xyz="1 0 0"/>
       <limit effort="130" lower="0" upper="0.025" velocity="0.15"/>
     </joint>
     <joint name="${prefix}robotiq_hand_e_right_finger_joint" type="prismatic">
-      <origin xyz="0 0 ${0.099 + 0.047}" rpy="0 0 0"/>
+      <origin xyz="0.025 0 ${0.099 + 0.047}" rpy="0 0 0"/>
       <parent link="${prefix}robotiq_hand_e_base_link"/>
       <child link="${prefix}robotiq_hand_e_right_finger"/>
-      <axis xyz="1 0 0"/>
+      <axis xyz="-1 0 0"/>
       <limit effort="130" lower="0" upper="0.025" velocity="0.15"/>
       <mimic joint="${prefix}robotiq_hand_e_left_finger_joint" multiplier="1" offset="0"/>
