Commit message: adjust srdf

File: robotiq_description/srdf/hand_e/hand_e_macro.srdf.xacro (robot description, xacro)
@@ -12,10 +12,11 @@
         </group_state>
         <group_state name="${prefix}close" group="${prefix}${name}_gripper">
-                <joint name="${prefix}robotiq_hand_e_left_finger_joint" value="-0.1"/>
-                <joint name="${prefix}robotiq_hand_e_right_finger_joint" value="0.1"/>
+                <joint name="${prefix}robotiq_hand_e_left_finger_joint" value="0.025"/>
+                <joint name="${prefix}robotiq_hand_e_right_finger_joint" value="0.025"/>
         </group_state>
         <disable_collisions link1="${prefix}robotiq_hand_e_base_link" link2="${prefix}link7" reason="Adjacent"/>
         <disable_collisions link1="${prefix}robotiq_hand_e_base_link" link2="${prefix}robotiq_hand_e_left_finger" reason="Adjacent"/>
         <disable_collisions link1="${prefix}robotiq_hand_e_base_link" link2="${prefix}robotiq_hand_e_right_finger" reason="Adjacent"/>
+        <disable_collisions link1="${prefix}robotiq_hand_e_left_finger" link2="${prefix}robotiq_hand_e_right_finger" reason="Never"/>
     </xacro:macro>
 </robot>

Commit message: when instantiating srdf, chose link to disable collisions for

File: robotiq_description/srdf/hand_e/hand_e_macro.srdf.xacro (robot description, xacro)
@@ -1,5 +1,5 @@
 <?xml version="1.0" encoding="UTF-8"?>
 <robot xmlns:xacro="http://www.ros.org/wiki/xacro">
-    <xacro:macro name="hand_e_srdf" params="name prefix">
+    <xacro:macro name="hand_e_srdf" params="name prefix disable_link_collision">
         <group name="${name}_gripper">
                 <link name="${prefix}robotiq_hand_e_base_link"/>
@@ -15,5 +15,5 @@
                 <joint name="${prefix}robotiq_hand_e_right_finger_joint" value="0.025"/>
         </group_state>
-        <disable_collisions link1="${prefix}robotiq_hand_e_base_link" link2="${prefix}link7" reason="Adjacent"/>
+        <disable_collisions link1="${prefix}robotiq_hand_e_base_link" link2="${prefix}${disable_link_collision}" reason="Adjacent"/>
         <disable_collisions link1="${prefix}robotiq_hand_e_base_link" link2="${prefix}robotiq_hand_e_left_finger" reason="Adjacent"/>
         <disable_collisions link1="${prefix}robotiq_hand_e_base_link" link2="${prefix}robotiq_hand_e_right_finger" reason="Adjacent"/>
